File: hardware/MCU.kicad_sch (KiCad schematic)
At the start: 13 parts, among them U202 STM32L431RCTx

Commit message: Adicionando arquivos do projeto
Changed lines of the file:
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@@
+		)
+	)
+	(hierarchical_label "Vcell3_stm"
+		(shape input)
+		(at 246.38 99.06 0)
+		(effects
+			(font
+				(size 1.27 1.27)
+			)
+			(justify left)
+		)
+	)
+	(hierarchical_label "Temp2_stm"
+		(shape input)
+		(at 246.38 107.696 0)
+		(effects
+			(font
+				(size 1.27 1.27)
+			)
+			(justify left)
+		)
+	)
+	(hierarchical_label "Temp3_stm"
+		(shape input)
+		(at 246.38 110.49 0)
+		(effects
+			(font
+				(size 1.27 1.27)
+			)
+			(justify left)
 		)
 	)
@@
 			(font
 				(size 1.016 1.016)
+			)
+			(justify left)
+		)
+	)
+	(hierarchical_label "Vcell2_stm"
+		(shape input)
+		(at 246.38 96.012 0)
+		(effects
+			(font
+				(size 1.27 1.27)
 			)
 			(justify left)
@@
 		)
 	)
+	(hierarchical_label "Vcell1_stm"
+		(shape input)
+		(at 246.38 93.218 0)
+		(effects
+			(font
+				(size 1.27 1.27)
+			)
+			(justify left)
+		)
+	)
 	(hierarchical_label "SWDIO"
 		(shape input)
@@
 			)
 			(justify left)
+		)
+	)
+	(hierarchical_label "Temp1_stm"
+		(shape input)
+		(at 246.38 104.648 0)
+		(effects
+			(font
+				(size 1.27 1.27)
+			)
+			(justify left)
+		)
+	)
+	(hierarchical_label "Vbanco_stm"
+		(shape input)
+		(at 246.38 101.854 0)
+		(effects
+			(font
+				(size 1.27 1.27)
+			)
+			(justify left)

Commit message: Atualização analog
Connections:
- net Temp1_stm: now also U202.20 (PA4)
- net Temp2_stm: now also U202.21 (PA5)
- net Temp3_stm: now also U202.22 (PA6)
- net Vbanco_stm: now also U202.17 (PA3)
- net Vcell1_stm: now also U202.14 (PA0)
- net Vcell2_stm: now also U202.15 (PA1)
- net Vcell3_stm: now also U202.16 (PA2)
- no-connect marks 15 -> 37
Changed lines of the file:
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@@
+	)
+	(no_connect
+		(at 167.64 121.92)
 	)
 	(no_connect
@@
 	)
 	(no_connect
+		(at 134.62 109.22)
+	)
+	(no_connect
+		(at 167.64 124.46)
+	)
+	(no_connect
+		(at 134.62 147.32)
+	)
+	(no_connect
 		(at 167.64 129.54)
 	)
 	(no_connect
+		(at 134.62 142.24)
+	)
+	(no_connect
 		(at 134.62 127)
 	)
@@
 	)
 	(no_connect
+		(at 167.64 144.78)
+	)
+	(no_connect
+		(at 167.64 83.82)
+	)
+	(no_connect
+		(at 167.64 127)
+	)
+	(no_connect
+		(at 134.62 124.46)
+	)
+	(no_connect
 		(at 134.62 137.16)
 	)
 	(no_connect
+		(at 167.64 119.38)
+	)
+	(no_connect
 		(at 167.64 134.62)
 	)
 	(no_connect
+		(at 167.64 86.36)
+	)
+	(no_connect
+		(at 134.62 116.84)
+	)
+	(no_connect
+		(at 167.64 142.24)
+	)
+	(no_connect
 		(at 134.62 134.62)
 	)
 	(no_connect
+		(at 134.62 114.3)
+	)
+	(no_connect
+		(at 134.62 121.92)
+	)
+	(no_connect
 		(at 134.62 132.08)
 	)
@@
 	)
 	(no_connect
+		(at 134.62 119.38)
+	)
+	(no_connect
 		(at 167.64 104.14)
 	)
 	(no_connect
+		(at 167.64 139.7)
+	)
+	(no_connect
+		(at 134.62 144.78)
+	)
+	(no_connect
+		(at 134.62 93.98)
+	)
+	(no_connect
 		(at 167.64 109.22)
 	)
 	(no_connect
+		(at 167.64 147.32)
+	)
+	(no_connect
 		(at 134.62 104.14)
 	)
+	(no_connect
+		(at 134.62 111.76)
+	)
+	(no_connect
+		(at 134.62 139.7)
+	)
 	(wire
 		(pts
@@
 	(wire
 		(pts
+			(xy 167.64 71.12) (xy 169.926 71.12)
+		)
+		(stroke
+			(width 0)
+			(type default)
+		)
+	)
+	(wire
+		(pts
 			(xy 188.722 27.178) (xy 188.722 30.988)
 		)
@@
 	(wire
 		(pts
+			(xy 167.64 81.28) (xy 169.926 81.28)
+		)
+		(stroke
+			(width 0)
+			(type default)
+		)
+	)
+	(wire
+		(pts
 			(xy 99.568 91.44) (xy 99.568 93.98)
 		)
@@
 		)
 	)
+	(wire
+		(pts
+			(xy 167.64 78.74) (xy 169.926 78.74)
+		)
+		(stroke
+			(width 0)
+			(type default)
+		)
+	)
 	(polyline
 		(pts
@@
 		)
 	)
+	(wire
+		(pts
+			(xy 167.64 76.2) (xy 169.926 76.2)
+		)
+		(stroke
+			(width 0)
+			(type default)
+		)
+	)
 	(polyline
 		(pts
@@
 	(wire
 		(pts
-			(xy 167.64 96.52) (xy 179.07 96.52)
+			(xy 167.64 96.52) (xy 169.926 96.52)
+		)
+		(stroke
+			(width 0)
+			(type default)
+		)
+	)
+	(wire
+		(pts
+			(xy 167.64 68.58) (xy 169.926 68.58)
 		)
 		(stroke
@@
 	(wire
 		(pts
-			(xy 167.64 116.84) (xy 182.88 116.84)
+			(xy 167.64 116.84) (xy 169.926 116.84)
 		)
 		(stroke
@@
 	(wire
 		(pts
-			(xy 167.64 93.98) (xy 179.07 93.98)
+			(xy 167.64 93.98) (xy 169.926 93.98)
 		)
 		(stroke
@@
 	(wire
 		(pts
-			(xy 167.64 88.9) (xy 182.88 88.9)
+			(xy 167.64 88.9) (xy 169.926 88.9)
 		)
 		(stroke
@@
 	(wire
 		(pts
-			(xy 167.64 101.6) (xy 182.245 101.6)
-		)
-		(stroke
-			(width 0)
-			(type default)
-		)
-	)
-	(wire
-		(pts
-			(xy 167.64 99.06) (xy 182.245 99.06)
+			(xy 167.64 101.6) (xy 169.926 101.6)
+		)
+		(stroke
+			(width 0)
+			(type default)
+		)
+	)
+	(wire
+		(pts
+			(xy 167.64 99.06) (xy 169.926 99.06)
 		)
 		(stroke
@@
 	(wire
 		(pts
-			(xy 167.64 91.44) (xy 182.88 91.44)
+			(xy 167.64 73.66) (xy 169.926 73.66)
+		)
+		(stroke
+			(width 0)
+			(type default)
+		)
+	)
+	(wire
+		(pts
+			(xy 167.64 91.44) (xy 169.926 91.44)
 		)
 		(stroke
@@
 		(pts
 			(xy 154.94 152.4) (xy 154.94 154.94)
+		)
+		(stroke
+			(width 0)
+			(type default)
+		)
+	)
+	(wire
+		(pts
+			(xy 167.64 66.04) (xy 169.926 66.04)
 		)
 		(stroke
@@
 	(hierarchical_label "Vcell3_stm"
 		(shape input)
-		(at 246.38 99.06 0)
+		(at 169.926 71.12 0)
 		(effects
 			(font
@@
 	(hierarchical_label "Temp2_stm"
 		(shape input)
-		(at 246.38 107.696 0)
+		(at 169.926 78.74 0)
 		(effects
 			(font
@@
 	(hierarchical_label "Temp3_stm"
 		(shape input)
-		(at 246.38 110.49 0)
+		(at 169.926 81.28 0)
 		(effects
 			(font
@@
 	(hierarchical_label "SWO"
 		(shape input)
-		(at 182.88 116.84 0)
+		(at 169.926 116.84 0)
 		(effects
 			(font
@@
 	(hierarchical_label "SWCLK"
 		(shape input)
-		(at 182.245 101.6 0)
+		(at 169.926 101.6 0)
 		(effects
 			(font
@@
 	(hierarchical_label "Vcell2_stm"
 		(shape input)
-		(at 246.38 96.012 0)
+		(at 169.926 68.58 0)
 		(effects
 			(font
@@
 	(hierarchical_label "USART_RX"
 		(shape input)
-		(at 182.88 91.44 0)
+		(at 169.926 91.44 0)
 		(effects
 			(font
@@
 	(hierarchical_label "CAN_RX"
 		(shape input)
-		(at 179.07 93.98 0)
+		(at 169.926 93.98 0)
 		(effects
 			(font
@@
 	(hierarchical_label "CAN_TX"
 		(shape input)
-		(at 179.07 96.52 0)
+		(at 169.926 96.52 0)
 		(effects
 			(font
@@
 	(hierarchical_label "Vcell1_stm"
 		(shape input)
-		(at 246.38 93.218 0)
+		(at 169.926 66.04 0)
 		(effects
 			(font
@@
 	(hierarchical_label "SWDIO"
 		(shape input)
-		(at 182.245 99.06 0)
+		(at 169.926 99.06 0)
 		(effects
 			(font
@@
 	(hierarchical_label "USART_TX"
 		(shape input)
-		(at 182.88 88.9 0)
+		(at 169.926 88.9 0)
 		(effects
 			(font
@@
 	(hierarchical_label "Temp1_stm"
 		(shape input)
-		(at 246.38 104.648 0)
+		(at 169.926 76.2 0)
 		(effects
 			(font
@@
 	(hierarchical_label "Vbanco_stm"
 		(shape input)
-		(at 246.38 101.854 0)
-		(effects
-			(font
+		(at 169.926 73.66 0)
+		(effects
+			(font

Commit message: Placa Finalizada para revisão
Connections:
- net GNDA is gone; now on net GND: C211.1, C213.1, U202.12 (VSSA)
- net Vcell1_stm: now also U202.15 (PA1); no longer U202.14 (PA0)
- net Vcell2_stm: now also U202.14 (PA0); no longer U202.15 (PA1)
- net I2C_2_SCL: now reaches U202.29 (PB10)
- net I2C_2_SDA: now reaches U202.30 (PB11)
- net I2C_1_SCL: now reaches U202.58 (PB6)
- net I2C_1_SDA: now reaches U202.59 (PB7)
- no-connect marks 37 -> 33
Changed lines of the file:
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@@
-	)
-	(no_connect
-		(at 167.64 137.16)
 	)
 	(no_connect
@@
 	)
 	(no_connect
-		(at 167.64 124.46)
-	)
-	(no_connect
 		(at 134.62 147.32)
 	)
@@
 	)
 	(no_connect
-		(at 167.64 127)
-	)
-	(no_connect
 		(at 134.62 124.46)
 	)
@@
 	)
 	(no_connect
-		(at 167.64 134.62)
-	)
-	(no_connect
 		(at 167.64 86.36)
 	)
@@
 	(wire
 		(pts
+			(xy 167.64 137.16) (xy 169.926 137.16)
+		)
+		(stroke
+			(width 0)
+			(type default)
+		)
+	)
+	(wire
+		(pts
 			(xy 157.48 44.196) (xy 157.48 45.212)
 		)
@@
 		)
 	)
+	(wire
+		(pts
+			(xy 167.64 124.46) (xy 169.926 124.46)
+		)
+		(stroke
+			(width 0)
+			(type default)
+		)
+	)
 	(polyline
 		(pts
@@
 	(wire
 		(pts
+			(xy 167.64 134.62) (xy 169.926 134.62)
+		)
+		(stroke
+			(width 0)
+			(type default)
+		)
+	)
+	(wire
+		(pts
 			(xy 123.825 42.545) (xy 149.86 42.545)
+		)
+		(stroke
+			(width 0)
+			(type default)
+		)
+	)
+	(wire
+		(pts
+			(xy 167.64 127) (xy 169.926 127)
 		)
 		(stroke
@@
 		)
 	)
+	(hierarchical_label "I2C_2_SDA"
+		(shape input)
+		(at 169.926 137.16 0)
+		(effects
+			(font
+				(size 1.27 1.27)
+			)
+			(justify left)
+		)
+	)
+	(hierarchical_label "I2C_1_SCL"
+		(shape input)
+		(at 169.926 124.46 0)
+		(effects
+			(font
+				(size 1.27 1.27)
+			)
+			(justify left)
+		)
+	)
 	(hierarchical_label "Temp3_stm"
 		(shape input)
@@
 		)
 	)
-	(hierarchical_label "Vcell2_stm"
+	(hierarchical_label "Vcell1_stm"
 		(shape input)
 		(at 169.926 68.58 0)
@@
 		)
 	)
+	(hierarchical_label "I2C_1_SDA"
+		(shape input)
+		(at 169.926 127 0)
+		(effects
+			(font
+				(size 1.27 1.27)
+			)
+			(justify left)
+		)
+	)
 	(hierarchical_label "USART_RX"
 		(shape input)
@@
 		)
 	)
-	(hierarchical_label "Vcell1_stm"
+	(hierarchical_label "Vcell2_stm"
 		(shape input)
 		(at 169.926 66.04 0)
@@
 		(shape input)
 		(at 169.926 76.2 0)
+		(effects
+			(font
+				(size 1.27 1.27)
+			)
+			(justify left)
+		)
+	)
+	(hierarchical_label "I2C_2_SCL"
+		(shape input)
+		(at 169.926 134.62 0)
 		(effects
 			(font
@@
 			)
 		)
-		(property "Value" "GNDA"
-			(at 154.94 159.3834 0)
+		(property "Value" "GND"
+			(at 154.94 160.02 0)
 			(effects
 				(font
@@
 			)
 		)
-		(property "Value" "GNDA"
+		(property "Value" "GND"
 			(at 170.815 63.4984 0)
 			(effects
