File: hardware/MSG25.kicad_sch (KiCad schematic)
At the start: 17 parts, among them J1 Conn_01x02, J101 USART, J102 STLink, J2 Conn_01x02, J3 Conn_01x02, J4 Conn_01x02, J5 Conn_01x02, J6 Conn_01x02, J7 Conn_01x02

Commit message: Adicionando arquivos do projeto
Connections:
- net GND: now also J1.2 (Pin_2), J2.2 (Pin_2), J3.2 (Pin_2), J4.2 (Pin_2), J5.2 (Pin_2), J6.2 (Pin_2), J7.2 (Pin_2)
- net ANALOG/Vcell1: now reaches J1.1 (Pin_1)
- net ANALOG/Temp1: now reaches J5.1 (Pin_1)
- net ANALOG/Vcell2: now reaches J2.1 (Pin_1)
- net ANALOG/Vbanco: now reaches J4.1 (Pin_1)
- net ANALOG/Vcell3: now reaches J3.1 (Pin_1)
- net ANALOG/Temp2: now reaches J6.1 (Pin_1)
- net ANALOG/Temp3: now reaches J7.1 (Pin_1)
Other:
- sheet ANALOG ports: added Temp1, Temp1_a, Temp2, Temp2_a, Temp3, Temp3_a, Vbanco, Vbanco_a, Vcell1, Vcell1_a, Vcell2, Vcell2_a, Vcell3, Vcell3_a; removed none
- sheet MCU ports: added Temp1_stm, Temp2_stm, Temp3_stm, Vbanco_stm, Vcell1_stm, Vcell2_stm, Vcell3_stm; removed none

Commit message: Atualização analog
Other:
- sheet ANALOG ports: added 15V, GND; removed none
Changed lines of the file:
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@@
+	(wire
+		(pts
+			(xy 228.346 27.686) (xy 228.346 65.024)
+		)
+		(stroke
+			(width 0)
+			(type default)
+		)
+	)
 	(wire
 		(pts
@@
 	(wire
 		(pts
+			(xy 98.806 27.686) (xy 228.346 27.686)
+		)
+		(stroke
+			(width 0)
+			(type default)
+		)
+	)
+	(wire
+		(pts
 			(xy 58.166 23.876) (xy 64.516 23.876)
 		)
@@
 		(pts
 			(xy 199.136 92.71) (xy 217.17 92.71)
+		)
+		(stroke
+			(width 0)
+			(type default)
+		)
+	)
+	(wire
+		(pts
+			(xy 231.14 64.008) (xy 231.14 65.024)
 		)
 		(stroke
@@
 	(symbol
 		(lib_id "power:GND")
+		(at 231.14 64.008 180)
+		(unit 1)
+		(exclude_from_sim no)
+		(in_bom yes)
+		(on_board yes)
+		(dnp no)
+		(fields_autoplaced yes)
+		(property "Reference" "#PWR015"
+			(at 231.14 57.658 0)
+			(effects
+				(font
+					(size 1.27 1.27)
+				)
+				(hide yes)
+			)
+		)
+		(property "Value" "GND"
+			(at 231.14 59.436 0)
+			(effects
+				(font
+					(size 1.27 1.27)
+				)
+			)
+		)
+		(property "Footprint" ""
+			(at 231.14 64.008 0)
+			(effects
+				(font
+					(size 1.27 1.27)
+				)
+				(hide yes)
+			)
+		)
+		(property "Datasheet" ""
+			(at 231.14 64.008 0)
+			(effects
+				(font
+					(size 1.27 1.27)
+				)
+				(hide yes)
+			)
+		)
+		(property "Description" "Power symbol creates a global label with name \"GND\" , ground"
+			(at 231.14 64.008 0)
+			(effects
+				(font
+					(size 1.27 1.27)
+				)
+				(hide yes)
+			)
+		)
+		(pin "1"
+		)
+		(instances
+			(project "MSG25"
+				(path "/65407f14-222c-4907-8176-906911332438"
+					(reference "#PWR015")
+					(unit 1)
+				)
+			)
+		)
+	)
+	(symbol
+		(lib_id "power:GND")
 		(at 70.866 26.416 0)
 		(unit 1)
@@
 			)
 		)
+		(pin "15V" input
+			(at 228.346 65.024 90)
+			(effects
+				(font
+					(size 1.27 1.27)
+				)
+				(justify right)
+			)
+		)
+		(pin "GND" input
+			(at 231.14 65.024 90)
+			(effects
+				(font
+					(size 1.27 1.27)
+				)
+				(justify right)
+			)
+		)

Commit message: Atualização analog
Connections:
- net GND: no longer J1.2 (Pin_2), J2.2 (Pin_2), J3.2 (Pin_2), J4.2 (Pin_2)
- net ANALOG/Vbanco renamed ANALOG/Vbanco+
- net ANALOG/Vcell1 renamed ANALOG/Vcell1+
- net ANALOG/Vcell2 renamed ANALOG/Vcell2+
- net ANALOG/Vcell3 renamed ANALOG/Vcell3+
- new net ANALOG/Vbanco-: J4.2 (Pin_2)
- new net ANALOG/Vcell1-: J1.2 (Pin_2)
- new net ANALOG/Vcell2-: J2.2 (Pin_2)
- new net ANALOG/Vcell3-: J3.2 (Pin_2)
Other:
- sheet ANALOG ports: added Vbanco+, Vbanco-, Vcell1+, Vcell1-, Vcell2+, Vcell2-, Vcell3+, Vcell3-; removed Vbanco, Vcell1, Vcell2, Vcell3

Commit message: Placa Finalizada para revisão
Parts:
- added J8: I2C_1, Connector_PinSocket_2.54mm:PinSocket_1x04_P2.54mm_Horizontal, symbol Connector_Generic:Conn_01x04
- added J9: I2C_2, Connector_PinSocket_2.54mm:PinSocket_1x04_P2.54mm_Horizontal, symbol Connector_Generic:Conn_01x04
- added LOGO101: Logo_Open_Hardware_Small, Symbol:OSHW-Logo2_7.3x6mm_SilkScreen, symbol Graphic:Logo_Open_Hardware_Small
- added R35, R36, R37, R38: 4k7, Resistor_SMD:R_0805_2012Metric_Pad1.20x1.40mm_HandSolder, symbol Device:R
- added SYM101, SYM102: SYM_Radioactive_Radiation_Small, KicadZeniteSolarLibrary18:symbol_logoZenite, symbol Graphic:SYM_Radioactive_Radiation_Small
- added SYM103: SYM_Radioactive_Radiation_Small, KicadZeniteSolarLibrary18:symbol_naolavar, symbol Graphic:SYM_Radioactive_Radiation_Small
- added SYM104, SYM105: SYM_LASER_Small, KicadZeniteSolarLibrary18:synbol_logoifsc, symbol Graphic:SYM_LASER_Small
- +Banco1-1: renamed from J4; footprint (none) -> TerminalBlock:TerminalBlock_bornier-2_P5.08mm
- -Temp1+1: renamed from J5; footprint (none) -> TerminalBlock:TerminalBlock_bornier-2_P5.08mm
- -Temp2+1: renamed from J6; footprint (none) -> TerminalBlock:TerminalBlock_bornier-2_P5.08mm
- -Temp3+1: renamed from J7; footprint (none) -> TerminalBlock:TerminalBlock_bornier-2_P5.08mm
- Cell1: renamed from J1; footprint (none) -> TerminalBlock:TerminalBlock_bornier-2_P5.08mm
- Cell2: renamed from J2; footprint (none) -> TerminalBlock:TerminalBlock_bornier-2_P5.08mm
- Cell3: renamed from J3; footprint (none) -> TerminalBlock:TerminalBlock_bornier-2_P5.08mm
- J101: footprint Connector_PinHeader_2.54mm:PinHeader_1x04_P2.54mm_Vertical_SMD_Pin1Left -> Connector_PinSocket_2.54mm:PinSocket_1x04_P2.54mm_Horizontal
- J102: footprint Connector_PinHeader_2.54mm:PinHeader_1x05_P2.54mm_Vertical_SMD_Pin1Left -> Connector_PinSocket_2.54mm:PinSocket_1x05_P2.54mm_Vertical
Connections:
- net +3V3: now also J8.3 (Pin_3), J9.3 (Pin_3), R35.2, R36.1, R37.2, R38.1
- net GND: now also J8.4 (Pin_4), J9.4 (Pin_4)
- new net MCU/I2C_1_SCL: J9.1 (Pin_1), R37.1
- new net MCU/I2C_1_SDA: J9.2 (Pin_2), R38.2
- new net MCU/I2C_2_SCL: J8.1 (Pin_1), R35.1
- new net MCU/I2C_2_SDA: J8.2 (Pin_2), R36.2
Other:
- sheet CANBUS ports: added +5V; removed 5v
- sheet MCU ports: added I2C_1_SCL, I2C_1_SDA, I2C_2_SCL, I2C_2_SDA; removed none
- moved on the sheet: C101, D108, D109, F101, H101, H102, H103, H104, J101, J102
