File: hardware/canbus.kicad_sch (KiCad schematic)
At the start: 13 parts, among them U501 MCP2561-E-SN

Commit message: Placa Finalizada para revisão
Parts:
- removed TP501: TxCAN, TestPoint:TestPoint_Pad_2.0x2.0mm, symbol Connector:TestPoint
- removed TP502: RxCAN, TestPoint:TestPoint_Pad_2.0x2.0mm, symbol Connector:TestPoint
- removed TP503: CAN_H, TestPoint:TestPoint_Pad_2.0x2.0mm, symbol Connector:TestPoint
- removed TP504: CAN_L, TestPoint:TestPoint_Pad_2.0x2.0mm, symbol Connector:TestPoint
Connections:
- net 5v renamed +5V
